File: v1.0/KiCAD/Toolbox_v1.0/Toolbox_v1.0.kicad_pcb (KiCad board)
At the start: 2 copper layers, 80.9 x 128.5 mm, 338 parts, among them J1 POWER, J10 Links_1to3_OUT1, J11 Links_1to3_IN, J12 Links_1to3_OUT2, J13 Links_1to3_OUT3, J14 Links_2to2_IN1, J15 Links_2to2_IN2, J16 Links_2to2_OUT1, J17 Links_2to2_OUT2, J18 Links_3to1_IN1, J19 Links_3to1_IN2, J2 OUT_1, J20 Links_3to1_OUT, J21 Links_3to1_IN3, J22 Kinks_IN, J23 Kinks_OUT_INV, J24 Kinks_OUT_HW, J25 Kinks_OUT_FW, J26 Kinks_OUT_MAX, J27 Kinks_IN_A, J28 Kinks_IN_B, J29 Kinks_OUT_MIN, J3 IN_1, J30 Kinks_OUT_Noise, J31 Kinks_OUT_S&H, J32 Kinks_S&H_IN, J33 Kinks_S&H_TRIG, J34 OUT_+10V, J35 IN_±5V, J36 IN_+10V, J37 OUT_±5V, J38 IN, J39 OUT_x1.25, J4 OUT_2, J40 OUT_x1.6, J41 OUT_x2, J5 IN_2, J6 OUT_3, J7 IN_3, J8 OUT_4, J9 IN_4, Q1 MMBT3904, Q2 MMBT3904, Q3 MMBFJ310, SW1 SW_SPDT, SW2 SW_SPDT, SW3 SW_SPDT, SW4 SW_SPDT, SW5 SW_SPDT, SW6 SW_SPDT, SW7 SW_SPDT, SW8 SW_SPDT, U1 TL074, U10 TL074, U11 TL074, U12 TL074, U13 CJ431, U14 CJ431, U15 CJ431, U2 TL074, U3 TL074, U4 TL074, U5 TL074, U6 TL074, U7 TL074, U8 TL074, U9 TL074

Commit message: v2.1 Update
Parts:
- R1, R4, R9: value 100R -> 1K
- R93: value 1.5M -> 240K
Other:
- board text added: "StduioKAT Toolbox v1.1 Inspired by Mutable Instruments Shades,Links,Kinks"
- board text removed: "StduioKAT Toolbox v1.0 Inspired by Mutable Instruments Shades,Links,Kinks"
