File: v2.1/KiCAD/Toolbox_v2.1/Kinks_2.kicad_sch (KiCad schematic)
At the start: 22 parts, among them J26 Kinks_OUT_MAX, J27 Kinks_IN_A, J28 Kinks_IN_B, J29 Kinks_OUT_MIN, U6 TL074, U7 TL074

Commit message: v2.1 Update
Parts:
- U6, U7: value TL074 -> TL074CDR; footprint Package_SO:TSSOP-14_4.4x5mm_P0.65mm -> Package_SO:SOIC-14_3.9x8.7mm_P1.27mm; LCSC C4370424 -> C12594
- renumbered R82 to R80, R83 to R81, R84 to R82, R85 to R83, R86 to R84, R87 to R85, R88 to R86, R89 to R87, R90 to R88
Changed lines of the file:
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@@
 	(title_block
 		(title "Analog AND/OR")
-		(date "2025-03-23")
-		(rev "1.0")
+		(date "2025-07-31")
+		(rev "2.1")
 		(company "StudioKAT")
 	)
@@
 		(on_board yes)
 		(dnp no)
-		(property "Reference" "#PWR082"
+		(property "Reference" "#PWR084"
 			(at 127 115.57 0)
 			(effects
@@
 			(project "Toolbox_1.3"
 				(path "/e7425001-019f-4fe8-a183-327e17dee003/8b736f3f-6587-48da-a243-a3526b0f68d8"
-					(reference "#PWR082")
+					(reference "#PWR084")
 					(unit 1)
 				)
@@
 		(dnp no)
 		(fields_autoplaced yes)
-		(property "Reference" "#PWR077"
+		(property "Reference" "#PWR079"
 			(at 93.98 54.61 0)
 			(effects
@@
 			(project "Toolbox_1.3"
 				(path "/e7425001-019f-4fe8-a183-327e17dee003/8b736f3f-6587-48da-a243-a3526b0f68d8"
-					(reference "#PWR077")
+					(reference "#PWR079")
 					(unit 1)
 				)
@@
 		(dnp no)
 		(fields_autoplaced yes)
-		(property "Reference" "R87"
+		(property "Reference" "R85"
 			(at 129.54 111.7599 0)
 			(effects
@@
 			(project "Toolbox_1.3"
 				(path "/e7425001-019f-4fe8-a183-327e17dee003/8b736f3f-6587-48da-a243-a3526b0f68d8"
-					(reference "R87")
+					(reference "R85")
 					(unit 1)
 				)
@@
 		(dnp no)
 		(fields_autoplaced yes)
-		(property "Reference" "#PWR076"
+		(property "Reference" "#PWR078"
 			(at 170.18 52.07 0)
 			(effects
@@
 			(project "Toolbox_1.3"
 				(path "/e7425001-019f-4fe8-a183-327e17dee003/8b736f3f-6587-48da-a243-a3526b0f68d8"
-					(reference "#PWR076")
+					(reference "#PWR078")
 					(unit 1)
 				)
@@
 		(dnp no)
 		(fields_autoplaced yes)
-		(property "Reference" "#PWR079"
+		(property "Reference" "#PWR081"
 			(at 93.98 80.01 0)
 			(effects
@@
 			(project "Toolbox_1.3"
 				(path "/e7425001-019f-4fe8-a183-327e17dee003/8b736f3f-6587-48da-a243-a3526b0f68d8"
-					(reference "#PWR079")
+					(reference "#PWR081")
 					(unit 1)
 				)
@@
 			)
 		)
-		(property "Value" "TL074"
+		(property "Value" "TL074CDR"
 			(at 140.97 101.6 0)
 			(effects
@@
 			)
 		)
-		(property "Footprint" "Package_SO:TSSOP-14_4.4x5mm_P0.65mm"
+		(property "Footprint" "Package_SO:SOIC-14_3.9x8.7mm_P1.27mm"
 			(at 139.7 96.52 0)
 			(effects
@@
 			)
 		)
-		(property "LCSC" "C4370424"
+		(property "LCSC" "C12594"
 			(at 140.97 93.98 0)
 			(effects
@@
 		(on_board yes)
 		(dnp no)
-		(property "Reference" "#PWR080"
+		(property "Reference" "#PWR082"
 			(at 119.38 82.55 0)
 			(effects
@@
 			(project "Toolbox_1.3"
 				(path "/e7425001-019f-4fe8-a183-327e17dee003/8b736f3f-6587-48da-a243-a3526b0f68d8"
-					(reference "#PWR080")
+					(reference "#PWR082")
 					(unit 1)
 				)
@@
 		(dnp no)
 		(fields_autoplaced yes)
-		(property "Reference" "R82"
+		(property "Reference" "R80"
 			(at 123.19 21.59 90)
 			(effects
@@
 			(project "Toolbox_1.3"
 				(path "/e7425001-019f-4fe8-a183-327e17dee003/8b736f3f-6587-48da-a243-a3526b0f68d8"
-					(reference "R82")
+					(reference "R80")
 					(unit 1)
 				)
@@
 		(dnp no)
 		(fields_autoplaced yes)
-		(property "Reference" "R88"
+		(property "Reference" "R86"
 			(at 123.19 133.35 90)
 			(effects
@@
 			(project "Toolbox_1.3"
 				(path "/e7425001-019f-4fe8-a183-327e17dee003/8b736f3f-6587-48da-a243-a3526b0f68d8"
-					(reference "R88")
+					(reference "R86")
 					(unit 1)
 				)
@@
 			)
 		)
-		(property "Value" "TL074"
+		(property "Value" "TL074CDR"
 			(at 140.97 46.99 0)
 			(effects
@@
 			)
 		)
-		(property "Footprint" "Package_SO:TSSOP-14_4.4x5mm_P0.65mm"
+		(property "Footprint" "Package_SO:SOIC-14_3.9x8.7mm_P1.27mm"
 			(at 139.7 41.91 0)
 			(effects
@@
 			)
 		)
-		(property "LCSC" "C4370424"
+		(property "LCSC" "C12594"
 			(at 140.97 39.37 0)
 			(effects
@@
 		(dnp no)
 		(fields_autoplaced yes)
-		(property "Reference" "R83"
+		(property "Reference" "R81"
 			(at 160.02 33.02 90)
 			(effects
@@
 			(project "Toolbox_1.3"
 				(path "/e7425001-019f-4fe8-a183-327e17dee003/8b736f3f-6587-48da-a243-a3526b0f68d8"
-					(reference "R83")
+					(reference "R81")
 					(unit 1)
 				)
@@
 		(on_board yes)
 		(dnp no)
-		(property "Reference" "#PWR078"
+		(property "Reference" "#PWR080"
 			(at 127 60.96 0)
 			(effects
@@
 			(project "Toolbox_1.3"
 				(path "/e7425001-019f-4fe8-a183-327e17dee003/8b736f3f-6587-48da-a243-a3526b0f68d8"
-					(reference "#PWR078")
+					(reference "#PWR080")
 					(unit 1)
 				)
@@
 			)
 		)
-		(property "Value" "TL074"
+		(property "Value" "TL074CDR"
 			(at 140.97 144.78 0)
 			(effects
@@
 			)
 		)
-		(property "Footprint" "Package_SO:TSSOP-14_4.4x5mm_P0.65mm"
+		(property "Footprint" "Package_SO:SOIC-14_3.9x8.7mm_P1.27mm"
 			(at 139.7 149.86 0)
 			(effects
@@
 			)
 		)
-		(property "LCSC" "C4370424"
+		(property "LCSC" "C12594"
 			(at 140.97 152.4 0)
 			(effects
@@
 		(dnp no)
 		(fields_autoplaced yes)
-		(property "Reference" "R90"
+		(property "Reference" "R88"
 			(at 123.19 166.37 90)
 			(effects
@@
 			(project "Toolbox_1.3"
 				(path "/e7425001-019f-4fe8-a183-327e17dee003/8b736f3f-6587-48da-a243-a3526b0f68d8"
-					(reference "R90")
+					(reference "R88")
 					(unit 1)
 				)
@@
 		(dnp no)
 		(fields_autoplaced yes)
-		(property "Reference" "R89"
+		(property "Reference" "R87"
 			(at 123.19 143.51 90)
 			(effects
@@
 			(project "Toolbox_1.3"
 				(path "/e7425001-019f-4fe8-a183-327e17dee003/8b736f3f-6587-48da-a243-a3526b0f68d8"
-					(reference "R89")
+					(reference "R87")
 					(unit 1)
 				)
@@
 		(dnp no)
 		(fields_autoplaced yes)
-		(property "Reference" "#PWR081"
+		(property "Reference" "#PWR083"
 			(at 170.18 106.68 0)
 			(effects
@@
 			(project "Toolbox_1.3"
 				(path "/e7425001-019f-4fe8-a183-327e17dee003/8b736f3f-6587-48da-a243-a3526b0f68d8"
-					(reference "#PWR081")
+					(reference "#PWR083")
 					(unit 1)
 				)
@@
 		(dnp no)
 		(fields_autoplaced yes)
-		(property "Reference" "R84"
+		(property "Reference" "R82"
 			(at 129.54 57.1499 0)
 			(effects
@@
 			(project "Toolbox_1.3"
 				(path "/e7425001-019f-4fe8-a183-327e17dee003/8b736f3f-6587-48da-a243-a3526b0f68d8"
-					(reference "R84")
+					(reference "R82")
 					(unit 1)
 				)
@@
 		(dnp no)
 		(fields_autoplaced yes)
-		(property "Reference" "R86"
+		(property "Reference" "R84"
 			(at 160.02 87.63 90)
 			(effects
@@
 			(project "Toolbox_1.3"
 				(path "/e7425001-019f-4fe8-a183-327e17dee003/8b736f3f-6587-48da-a243-a3526b0f68d8"
-					(reference "R86")
+					(reference "R84")
 					(unit 1)
 				)
@@
 		(dnp no)
 		(fields_autoplaced yes)
-		(property "Reference" "#PWR083"
+		(property "Reference" "#PWR085"
 			(at 116.84 181.61 0)
 			(effects
@@
 			(project "Toolbox_1.3"
 				(path "/e7425001-019f-4fe8-a183-327e17dee003/8b736f3f-6587-48da-a243-a3526b0f68d8"
-					(reference "#PWR083")
+					(reference "#PWR085")
 					(unit 1)
 				)
@@
 		(on_board yes)
 		(dnp no)
-		(property "Reference" "#PWR075"
+		(property "Reference" "#PWR077"
 			(at 119.38 27.94 0)
 			(effects
@@
 			(project "Toolbox_1.3"
 				(path "/e7425001-019f-4fe8-a183-327e17dee003/8b736f3f-6587-48da-a243-a3526b0f68d8"
-					(reference "#PWR075")
+					(reference "#PWR077")
 					(unit 1)
 				)
@@
 		(dnp no)
 		(fields_autoplaced yes)
-		(property "Reference" "R85"
+		(property "Reference" "R83"
 			(at 123.19 76.2 90)
 			(effects
@@
 			(project "Toolbox_1.3"
 				(path "/e7425001-019f-4fe8-a183-327e17dee003/8b736f3f-6587-48da-a243-a3526b0f68d8"
-					(reference "R85")
+					(reference "R83")
 					(unit 1)
 				)
