File: v2.1/KiCAD/Toolbox_v2.1/Shades.kicad_sch (KiCad schematic)
At the start: 69 parts, among them J2 OUT_1, J3 IN_1, J4 OUT_2, J5 IN_2, J6 OUT_3, J7 IN_3, J8 OUT_4, J9 IN_4, SW1 SW_SPDT, SW2 SW_SPDT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

Commit message: v2.1 Update
Parts:
- U1, U2, U3, U4: value TL074 -> TL074CDR; footprint Package_SO:TSSOP-14_4.4x5mm_P0.65mm -> Package_SO:SOIC-14_3.9x8.7mm_P1.27mm; LCSC C4370424 -> C12594
- renumbered C35 to C33, C36 to C34, C37 to C35, C38 to C36, R12 to R10, R13 to R11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
