File: v2.1/KiCAD/Toolbox_v2.1/Toolbox_v2.1.kicad_pcb (KiCad board)
At the start: 2 copper layers, 80.9 x 128.5 mm, 340 parts, among them J1 POWER, J10 Links_1to3_OUT1, J11 Links_1to3_IN, J12 Links_3to1_IN1, J13 Links_1to3_OUT2, J14 Links_3to1_IN2, J15 Links_3to1_OUT, J16 Links_1to3_OUT3, J17 Links_3to1_IN3, J18 Links_2to2_IN1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

Commit message: R91 定数変更 240K→200K
Parts:
- R91: value 240K -> 200K
