File: v2.1/KiCAD/Toolbox_v2.1/Voltage_Doubler.kicad_sch (KiCad schematic)
At the start: 21 parts, among them J38 IN, J39 OUT_x1.25, J40 OUT_x1.6, J41 OUT_x2, U12 TL074, U4 TL074, U8 TL074

Commit message: v2.1 Update
Parts:
- U12, U4, U8: value TL074 -> TL074CDR; footprint Package_SO:TSSOP-14_4.4x5mm_P0.65mm -> Package_SO:SOIC-14_3.9x8.7mm_P1.27mm; LCSC C4370424 -> C12594
- renumbered J38 to J39, J39 to J40, J40 to J41, J41 to J42, R118 to R119, R119 to R120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
